Commit message: feat(lekiwi): 添加集成底盘控制器并重构机器人配置
- 添加新的 base_controller.py 脚本，集成了运动控制和里程计算法
- 从 CMakeLists.txt 中移除 test_odometry.py 并添加 base_controller.py 到安装脚本
- 修改 launch 文件以使用新的 base_controller.py 替代 holonomic_controller.py
- 重命名 launch 文件中的节点名称从 holonomic_controller 到 base_controller
- 更新配置文件 controllers.yaml 移除不必要的关节状态广播器和服务端口配置
- 修改 URDF 文件修复后轮和右轮的链接配置
- 优化 C++ 代码中的速度读取逻辑和状态初始化
- 更新里程计发布脚本以基于命令输入进行调试模式运行
```

File: src/lekiwi/urdf/lekiwi_base.urdf (robot description, URDF)
Before this commit: robot lekiwi, 2 links, 3 joints
Links:
- added link rear_wheel_link; visual cylinder length=0.02 radius=0.03
- added link right_wheel_link; visual cylinder length=0.02 radius=0.03
Joints:
- joint rear_wheel_drive: child left_wheel_link -> rear_wheel_link
- joint right_wheel_drive: child left_wheel_link -> right_wheel_link
