Commit message: Refactor code structure for improved readability and maintainability

File: src/lekiwi/urdf/lekiwi_isaacsim copy.urdf (robot description, URDF)
Before this commit: robot lekiwi, 20 links, 19 joints
Links:
- removed link Omni_Directional_Wheel_Single_Body_v1
- removed link Omni_Directional_Wheel_Single_Body_v1_1
- removed link Omni_Directional_Wheel_Single_Body_v1_2
- removed link pillar_standoff
- removed link pillar_standoff_1
- removed link pillar_standoff_2
- removed link pillar_standoff_3
- removed link pillar_standoff_4
- removed link pillar_standoff_5
- added link 4_Omni_Directional_Wheel_Single_Body_v1, mass 1.3542854082324305; collision mesh filename=file:///home/synapath/workspase/ros2_lekiwi_classis/src/lek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 scale=0.001 0.001 0.001; visual mesh filename=file:///home/synapath/workspase/ros2_lekiwi_classis/src/lek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 scale=0.001 0.001 0.001
- added link 4_Omni_Directional_Wheel_Single_Body_v1_1, mass 1.3542854082324305; collision mesh filename=file:///home/synapath/workspase/ros2_lekiwi_classis/src/lek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 scale=0.001 0.001 0.001; visual mesh filename=file:///home/synapath/workspase/ros2_lekiwi_classis/src/lek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 scale=0.001 0.001 0.001
- added link 4_Omni_Directional_Wheel_Single_Body_v1_2, mass 1.3542854082324305; collision mesh filename=file:///home/synapath/workspase/ros2_lekiwi_classis/src/lek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 scale=0.001 0.001 0.001; visual mesh filename=file:///home/synapath/workspase/ros2_lekiwi_classis/src/lek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 scale=0.001 0.001 0.001
- added link 94868A713_NO_THREADS_Female_Threaded_Hex_Standoff, mass 0.006150070863406618; collision mesh filename=file:///home/synapath/workspase/ros2_lekiwi_classis/src/lek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 scale=0.001 0.001 0.001; visual mesh filename=file:///home/synapath/workspase/ros2_lekiwi_classis/src/lek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 scale=0.001 0.001 0.001
- added link 94868A713_NO_THREADS_Female_Threaded_Hex_Standoff_1, mass 0.006150070863406618; collision mesh filename=file:///home/synapath/workspase/ros2_lekiwi_classis/src/lek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 scale=0.001 0.001 0.001; visual mesh filename=file:///home/synapath/workspase/ros2_lekiwi_classis/src/lek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 scale=0.001 0.001 0.001
- added link 94868A713_NO_THREADS_Female_Threaded_Hex_Standoff_2, mass 0.006150070863406618; collision mesh filename=file:///home/synapath/workspase/ros2_lekiwi_classis/src/lek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 scale=0.001 0.001 0.001; visual mesh filename=file:///home/synapath/workspase/ros2_lekiwi_classis/src/lek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 scale=0.001 0.001 0.001
- added link 94868A713_NO_THREADS_Female_Threaded_Hex_Standoff_3, mass 0.006150070863406618; collision mesh filename=file:///home/synapath/workspase/ros2_lekiwi_classis/src/lek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 scale=0.001 0.001 0.001; visual mesh filename=file:///home/synapath/workspase/ros2_lekiwi_classis/src/lek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 scale=0.001 0.001 0.001
- added link 94868A713_NO_THREADS_Female_Threaded_Hex_Standoff_4, mass 0.006150070863406618; collision mesh filename=file:///home/synapath/workspase/ros2_lekiwi_classis/src/lek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 scale=0.001 0.001 0.001; visual mesh filename=file:///home/synapath/workspase/ros2_lekiwi_classis/src/lek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 scale=0.001 0.001 0.001
- added link 94868A713_NO_THREADS_Female_Threaded_Hex_Standoff_5, mass 0.006150070863406618; collision mesh filename=file:///home/synapath/workspase/ros2_lekiwi_classis/src/lek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 scale=0.001 0.001 0.001; visual mesh filename=file:///home/synapath/workspase/ros2_lekiwi_classis/src/lek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 scale=0.001 0.001 0.001
- link ST3215_Servo_Motor_v1: geometry collision mesh filename=file:///home/synapath/workspase/ros2_lekiwi_classis/src/lek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 scale=0.001 0.001 0.001; visual mesh filename=file:///home/synapath/workspase/ros2_lekiwi_classis/src/lek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 scale=0.001 0.001 0.001
- link ST3215_Servo_Motor_v1_1: geometry collision mesh filename=file:///home/synapath/workspase/ros2_lekiwi_classis/src/lek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 scale=0.001 0.001 0.001; visual mesh filename=file:///home/synapath/workspase/ros2_lekiwi_classis/src/lek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 scale=0.001 0.001 0.001
- link ST3215_Servo_Motor_v1_2: geometry collision mesh filename=file:///home/synapath/workspase/ros2_lekiwi_classis/src/lek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 scale=0.001 0.001 0.001; visual mesh filename=file:///home/synapath/workspase/ros2_lekiwi_classis/src/lek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 scale=0.001 0.001 0.001
- link base_link: geometry collision mesh filename=file:///home/synapath/workspase/ros2_lekiwi_classis/src/lek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 scale=0.001 0.001 0.001; visual mesh filename=file:///home/synapath/workspase/ros2_lekiwi_classis/src/lek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 scale=0.001 0.001 0.001
- link base_plate_layer2_v3: geometry collision mesh filename=file:///home/synapath/workspase/ros2_lekiwi_classis/src/lek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 scale=0.001 0.001 0.001; visual mesh filename=file:///home/synapath/workspase/ros2_lekiwi_classis/src/lek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 scale=0.001 0.001 0.001
- link drive_motor_mount_v11: geometry collision mesh filename=file:///home/synapath/workspase/ros2_lekiwi_classis/src/lek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 scale=0.001 0.001 0.001; visual mesh filename=file:///home/synapath/workspase/ros2_lekiwi_classis/src/lek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 scale=0.001 0.001 0.001
- link drive_motor_mount_v11_1: geometry collision mesh filename=file:///home/synapath/workspase/ros2_lekiwi_classis/src/lek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 scale=0.001 0.001 0.001; visual mesh filename=file:///home/synapath/workspase/ros2_lekiwi_classis/src/lek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 scale=0.001 0.001 0.001
- link drive_motor_mount_v11_2: geometry collision mesh filename=file:///home/synapath/workspase/ros2_lekiwi_classis/src/lek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 scale=0.001 0.001 0.001; visual mesh filename=file:///home/synapath/workspase/ros2_lekiwi_classis/src/lek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 scale=0.001 0.001 0.001
- link omni_wheel_mount_v5: geometry collision mesh filename=file:///home/synapath/workspase/ros2_lekiwi_classis/src/lek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 scale=0.001 0.001 0.001; visual mesh filename=file:///home/synapath/workspase/ros2_lekiwi_classis/src/lek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 scale=0.001 0.001 0.001
- link omni_wheel_mount_v5_1: geometry collision mesh filename=file:///home/synapath/workspase/ros2_lekiwi_classis/src/lek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 scale=0.001 0.001 0.001; visual mesh filename=file:///home/synapath/workspase/ros2_lekiwi_classis/src/lek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 scale=0.001 0.001 0.001
- link omni_wheel_mount_v5_2: geometry collision mesh filename=file:///home/synapath/workspase/ros2_lekiwi_classis/src/lek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 scale=0.001 0.001 0.001; visual mesh filename=file:///home/synapath/workspase/ros2_lekiwi_classis/src/lek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 scale=0.001 0.001 0.001
Joints:
- removed joint pillar_standoff_Rigid_21
- added joint 94868A713_NO_THREADS_Female_Threaded_Hex_Standoff_Rigid_21: type fixed, parent 94868A713_NO_THREADS_Female_Threaded_Hex_Standoff, child base_plate_layer2_v3, origin xyz=0.0 0.0 -0.05 rpy=3.141592653589793 -0.0 0.0
- joint base_plate_layer1_v5_Rigid_20: child pillar_standoff -> 94868A713_NO_THREADS_Female_Threaded_Hex_Standoff
- joint base_plate_layer1_v5_Rigid_30: child pillar_standoff_5 -> 94868A713_NO_THREADS_Female_Threaded_Hex_Standoff_5
- joint base_plate_layer1_v5_Rigid_31: child pillar_standoff_4 -> 94868A713_NO_THREADS_Female_Threaded_Hex_Standoff_4
- joint base_plate_layer1_v5_Rigid_32: child pillar_standoff_3 -> 94868A713_NO_THREADS_Female_Threaded_Hex_Standoff_3
- joint base_plate_layer1_v5_Rigid_69: child pillar_standoff_2 -> 94868A713_NO_THREADS_Female_Threaded_Hex_Standoff_2
- joint base_plate_layer1_v5_Rigid_70: child pillar_standoff_1 -> 94868A713_NO_THREADS_Female_Threaded_Hex_Standoff_1
- joint omni_wheel_mount_v5_1_Rigid_63: child Omni_Directional_Wheel_Single_Body_v1_1 -> 4_Omni_Directional_Wheel_Single_Body_v1_1
- joint omni_wheel_mount_v5_2_Rigid_61: child Omni_Directional_Wheel_Single_Body_v1_2 -> 4_Omni_Directional_Wheel_Single_Body_v1_2
- joint omni_wheel_mount_v5_Rigid_65: child Omni_Directional_Wheel_Single_Body_v1 -> 4_Omni_Directional_Wheel_Single_Body_v1
