Commit message: Remove outdated URDF file for the lekiwi robot model, consolidating resources and improving project structure.

File: src/lekiwi/urdf/lekiwi.urdf (robot description, URDF)
Before this commit: robot lekiwi, 20 links, 19 joints
Links:
- added link robot_base_classis; collision mesh filename=package://lekiwi/models/lekiwi_mobile_base/meshes/base_plat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 scale=0.001 0.001 0.001; visual mesh filename=package://lekiwi/models/lekiwi_mobile_base/meshes/base_plat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 scale=0.001 0.001 0.001
- link base_link: geometry 
Joints:
- added joint base_link_joint: type fixed, parent base_link, child robot_base_classis, origin xyz=0.0 0.0 0.0 rpy=0.0 -0.0 4.7123889804
- joint base_plate_layer1_v5_Rigid_20: parent base_link -> robot_base_classis
- joint base_plate_layer1_v5_Rigid_30: parent base_link -> robot_base_classis
- joint base_plate_layer1_v5_Rigid_31: parent base_link -> robot_base_classis
- joint base_plate_layer1_v5_Rigid_32: parent base_link -> robot_base_classis
- joint base_plate_layer1_v5_Rigid_69: parent base_link -> robot_base_classis
- joint base_plate_layer1_v5_Rigid_70: parent base_link -> robot_base_classis
- joint base_plate_layer1_v5_baseplate2bottom_mount: parent base_link -> robot_base_classis
- joint base_plate_layer1_v5_baseplate2left_mount: parent base_link -> robot_base_classis
- joint base_plate_layer1_v5_baseplate2right_mount: parent base_link -> robot_base_classis

Commit message: 修改urdf符合USD配置

File: src/lekiwi/urdf/lekiwi.urdf (robot description, URDF)
Before this commit: robot lekiwi, 21 links, 20 joints
Links:
- link base_link: mass None -> 0.01
- link robot_base_classis: mass None -> 1.9153836917607525
